File: DCPower - Simple/Power.kicad_sch (KiCad schematic)
At the start: 73 parts, among them J1 USB_C_Receptacle_USB2.0_14P, Q4 DMP4025LSD-13, Q5 DMP4025LSD-13, Q6 2N7002, Q9 SQ2319CES-T1_GE3, U1 USBLC6-2SC6, U2 CYPD3177-24LQ, U3 LMR33630CDDA, U4 MCP1727T-3302E_SN

Commit message: Update
Parts:
- removed U1: USBLC6-2SC6, Package_TO_SOT_SMD:SOT-23-6, symbol Power_Protection:USBLC6-2SC6
Connections:
- net at J1.A7 (D-): no longer J1.B7 (D-)
- net at J1.A6 (D+): no longer J1.B6 (D+)
Other:
- moved on the sheet: C10, C11, C12, C13, C14, C17, C18, C19, C20, C21, C22, C23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
