File: DCPower - Simple/DCPower - Simple.kicad_sch (KiCad schematic)
At the start: 4 parts

Commit message: Update
Parts:
- added C1, C37, C38: 10nF, PCM_JLCPCB:C_0603, symbol PCM_JLCPCB-Capacitors:0603,10nF
- added C15, C4, C6: 100nF, PCM_JLCPCB:C_0603, symbol PCM_JLCPCB-Capacitors:0603,100nF
- added C16: 10uF, PCM_JLCPCB:C_1206, symbol PCM_JLCPCB-Capacitors:1206,10uF
- added C2, C33, C34, C35, C36: 22 uF, PCM_JLCPCB:C_1206, symbol Device:C
- added C5: 1uF, PCM_JLCPCB:C_0603, symbol PCM_JLCPCB-Capacitors:0603,1uF
- added L3: XAL7070-472ME, symbol Device:L
- added R10: 0Ω, PCM_JLCPCB:R_0603, symbol PCM_JLCPCB-Resistors:0603,0Ω
- added R4, R8: 10kΩ, PCM_JLCPCB:R_0603, symbol PCM_JLCPCB-Resistors:0603,10kΩ
- added R5, R6, R9: 24kΩ, PCM_JLCPCB:R_0603, symbol PCM_JLCPCB-Resistors:0603,24kΩ
- added R7: 10 mΩ, symbol Device:R
- added U1: TPS55287RYQR, TPS552892RYQR, symbol DCPower:TPS55287RYQR
Connections:
- net +3.3V: now also R8.1
- net +V_MAIN: now also C2.1, C4.1, C5.1, R5.1, U1.7 (VIN)
- net GND: now also C1.2, C16.1, C2.2, C33.2, C34.2, C35.2, C36.2, C37.2, C38.2, C4.2, C5.2, R10.2, R4.2, R6.2, U1.17 (AGND), U1.2 (MODE), U1.21 (EXTVCC), U1.22 (PGND_2), U1.23 (PGND_3), U1.9 (PGND_1)
- new net: R10.1, U1.16 (CDC)
- new net: C33.1, C34.1, C35.1, C36.1, R7.1, U1.11 (VOUT), U1.12 (ISP)
- new net: C6.1, L3.1, U1.8 (SW1)
- new net: C6.2, U1.20 (BOOT1)
- new net: R7.2, U1.13 (ISN)
- new net: R8.2, U1.14 (FB/~{INT})
- new net: R9.1, U1.15 (COMP)
- new net: C38.1, R9.2
- new net: R4.1, R5.2, U1.1 (EN/UVLO)
- new net: C1.1, C37.1, U1.5 (DITH/SYNC)
- new net: C15.1, L3.2, U1.10 (SW2)
- new net: C15.2, U1.19 (BOOT2)
- new net: R6.1, U1.6 (FSW)
- new net +5V: C16.2, U1.18 (VCC)
Other:
- note added: "0x75H"
- note added: "4.182 UVLO"
- note added: "811kHz SW 744 Hz Dith"

Commit message: Update
Other:
- note added: "0x75h"
- note removed: "0x75H"
Changed lines of the file:
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@@
 		)
 	)
-	(text "0x75H"
+	(text "0x75h"
 		(exclude_from_sim no)
 		(at 260.096 61.214 0)
